Commit message: Modify sensor config (#4)
* Update x1 sensor config files

Signed-off-by: wep21 <border_goldenmarket@yahoo.co.jp>

* Update xx1 sensor config files

Signed-off-by: wep21 <border_goldenmarket@yahoo.co.jp>

* Update x2 sensor config files

Signed-off-by: wep21 <border_goldenmarket@yahoo.co.jp>

* Run pre-commit

Signed-off-by: wep21 <border_goldenmarket@yahoo.co.jp>

* Add prettier-xacro to pre-commit (#6)

Signed-off-by: Kenji Miyake <kenji.miyake@tier4.jp>

* Run pre-commit

Signed-off-by: wep21 <border_goldenmarket@yahoo.co.jp>

* Update README.md

Signed-off-by: wep21 <border_goldenmarket@yahoo.co.jp>

* Fix for pre-commit

Signed-off-by: Kenji Miyake <kenji.miyake@tier4.jp>

* Cosmetic change

Signed-off-by: wep21 <border_goldenmarket@yahoo.co.jp>

* Add _link

Signed-off-by: wep21 <border_goldenmarket@yahoo.co.jp>

* Fix missing link

Co-authored-by: Kenji Miyake <31987104+kenji-miyake@users.noreply.github.com>
Co-authored-by: Kenji Miyake <kenji.miyake@tier4.jp>

File: aip_x1_description/urdf/sensor_kit.xacro (robot description, xacro)
@@ -17,11 +17,52 @@
     <xacro:property name="calibration" value="${load_yaml('$(arg config_dir)/sensor_kit_calibration.yaml')}"/>
     <!-- lidar -->
-    <xacro:VLP-16 parent="sensor_kit_base_link" name="velodyne_top" topic="/points_raw" hz="10" samples="220" gpu="$(arg gpu)">
-      <origin xyz="${calibration['sensor_kit_base_link2velodyne_top_base_link']['x']} ${calibration['sensor_kit_base_link2velodyne_top_base_link']['y']} ${calibration['sensor_kit_base_link2velodyne_top_base_link']['z']}" rpy="${calibration['sensor_kit_base_link2velodyne_top_base_link']['roll']} ${calibration['sensor_kit_base_link2velodyne_top_base_link']['pitch']} ${calibration['sensor_kit_base_link2velodyne_top_base_link']['yaw']}" />
+    <xacro:VLP-16
+      parent="sensor_kit_base_link"
+      name="velodyne_top"
+      topic="/points_raw"
+      hz="10"
+      samples="220"
+      gpu="$(arg gpu)"
+    >
+      <origin
+        xyz="${calibration['sensor_kit_base_link']['velodyne_top_base_link']['x']}
+             ${calibration['sensor_kit_base_link']['velodyne_top_base_link']['y']}
+             ${calibration['sensor_kit_base_link']['velodyne_top_base_link']['z']}"
+        rpy="${calibration['sensor_kit_base_link']['velodyne_top_base_link']['roll']}
+             ${calibration['sensor_kit_base_link']['velodyne_top_base_link']['pitch']}
+            ${calibration['sensor_kit_base_link']['velodyne_top_base_link']['yaw']}"
+      />
     </xacro:VLP-16>
     <xacro:include filename="$(find livox_description)/urdf/livox_horizon.xacro"/>
-    <xacro:livox_horizon_macro name="livox_front_left" parent="sensor_kit_base_link" x="${calibration['sensor_kit_base_link2livox_front_left_base_link']['x']}" y="${calibration['sensor_kit_base_link2livox_front_left_base_link']['y']}" z="${calibration['sensor_kit_base_link2livox_front_left_base_link']['z']}" roll="${calibration['sensor_kit_base_link2livox_front_left_base_link']['roll']}" pitch="${calibration['sensor_kit_base_link2livox_front_left_base_link']['pitch']}" yaw="${calibration['sensor_kit_base_link2livox_front_left_base_link']['yaw']}" />
-    <xacro:livox_horizon_macro name="livox_front_center" parent="sensor_kit_base_link" x="${calibration['sensor_kit_base_link2livox_front_center_base_link']['x']}" y="${calibration['sensor_kit_base_link2livox_front_center_base_link']['y']}" z="${calibration['sensor_kit_base_link2livox_front_center_base_link']['z']}" roll="${calibration['sensor_kit_base_link2livox_front_center_base_link']['roll']}" pitch="${calibration['sensor_kit_base_link2livox_front_center_base_link']['pitch']}" yaw="${calibration['sensor_kit_base_link2livox_front_center_base_link']['yaw']}" />
-    <xacro:livox_horizon_macro name="livox_front_right" parent="sensor_kit_base_link" x="${calibration['sensor_kit_base_link2livox_front_right_base_link']['x']}" y="${calibration['sensor_kit_base_link2livox_front_right_base_link']['y']}" z="${calibration['sensor_kit_base_link2livox_front_right_base_link']['z']}" roll="${calibration['sensor_kit_base_link2livox_front_right_base_link']['roll']}" pitch="${calibration['sensor_kit_base_link2livox_front_right_base_link']['pitch']}" yaw="${calibration['sensor_kit_base_link2livox_front_right_base_link']['yaw']}" />
+    <xacro:livox_horizon_macro
+      name="livox_front_left"
+      parent="sensor_kit_base_link"
+      x="${calibration['sensor_kit_base_link']['livox_front_left_base_link']['x']}"
+      y="${calibration['sensor_kit_base_link']['livox_front_left_base_link']['y']}"
+      z="${calibration['sensor_kit_base_link']['livox_front_left_base_link']['z']}"
+      roll="${calibration['sensor_kit_base_link']['livox_front_left_base_link']['roll']}"
+      pitch="${calibration['sensor_kit_base_link']['livox_front_left_base_link']['pitch']}"
+      yaw="${calibration['sensor_kit_base_link']['livox_front_left_base_link']['yaw']}"
+    />
+    <xacro:livox_horizon_macro
+      name="livox_front_center"
+      parent="sensor_kit_base_link"
+      x="${calibration['sensor_kit_base_link']['livox_front_center_base_link']['x']}"
+      y="${calibration['sensor_kit_base_link']['livox_front_center_base_link']['y']}"
+      z="${calibration['sensor_kit_base_link']['livox_front_center_base_link']['z']}"
+      roll="${calibration['sensor_kit_base_link']['livox_front_center_base_link']['roll']}"
+      pitch="${calibration['sensor_kit_base_link']['livox_front_center_base_link']['pitch']}"
+      yaw="${calibration['sensor_kit_base_link']['livox_front_center_base_link']['yaw']}"
+    />
+    <xacro:livox_horizon_macro
+      name="livox_front_right"
+      parent="sensor_kit_base_link"
+      x="${calibration['sensor_kit_base_link']['livox_front_right_base_link']['x']}"
+      y="${calibration['sensor_kit_base_link']['livox_front_right_base_link']['y']}"
+      z="${calibration['sensor_kit_base_link']['livox_front_right_base_link']['z']}"
+      roll="${calibration['sensor_kit_base_link']['livox_front_right_base_link']['roll']}"
+      pitch="${calibration['sensor_kit_base_link']['livox_front_right_base_link']['pitch']}"
+      yaw="${calibration['sensor_kit_base_link']['livox_front_right_base_link']['yaw']}"
+    />
   </xacro:macro>
 </robot>

File: aip_x1_description/urdf/sensors.xacro (robot description, xacro)
@@ -1,10 +1,17 @@
 <?xml version="1.0"?>
-<robot name="vehicle"
-  xmlns:xacro="http://ros.org/wiki/xacro">
+<robot name="vehicle" xmlns:xacro="http://ros.org/wiki/xacro">
   <xacro:arg name="config_dir" default="$(find aip_x1_description)/config"/>
   <xacro:include filename="$(find aip_x1_description)/urdf/sensor_kit.xacro"/>
   <xacro:property name="calibration" value="${load_yaml('$(arg config_dir)/sensors_calibration.yaml')}"/>
   <!-- sensor kit -->
-  <xacro:sensor_kit_macro parent="base_link" x="${calibration['base_link2sensor_kit_base_link']['x']}" y="${calibration['base_link2sensor_kit_base_link']['y']}" z="${calibration['base_link2sensor_kit_base_link']['z']}" roll="${calibration['base_link2sensor_kit_base_link']['roll']}" pitch="${calibration['base_link2sensor_kit_base_link']['pitch']}" yaw="${calibration['base_link2sensor_kit_base_link']['yaw']}" />
+  <xacro:sensor_kit_macro
+    parent="base_link"
+    x="${calibration['base_link']['sensor_kit_base_link']['x']}"
+    y="${calibration['base_link']['sensor_kit_base_link']['y']}"
+    z="${calibration['base_link']['sensor_kit_base_link']['z']}"
+    roll="${calibration['base_link']['sensor_kit_base_link']['roll']}"
+    pitch="${calibration['base_link']['sensor_kit_base_link']['pitch']}"
+    yaw="${calibration['base_link']['sensor_kit_base_link']['yaw']}"
+  />
   <!-- embedded sensors -->
 </robot>

File: aip_x2_description/urdf/front_unit.xacro (robot description, xacro)
@@ -18,18 +18,24 @@
     <xacro:property name="calibration" value="${load_yaml('$(arg config_dir)/front_unit_calibration.yaml')}"/>
     <!-- lidar -->
-    <xacro:Pandar40P name="pandar_40p_front" parent="front_unit_base_link"
-      x="${calibration['front_unit_base_link2pandar_40p_front_base_link']['x']}"
-      y="${calibration['front_unit_base_link2pandar_40p_front_base_link']['y']}"
-      z="${calibration['front_unit_base_link2pandar_40p_front_base_link']['z']}"
-      roll="${calibration['front_unit_base_link2pandar_40p_front_base_link']['roll']}"
-      pitch="${calibration['front_unit_base_link2pandar_40p_front_base_link']['pitch']}"
-      yaw="${calibration['front_unit_base_link2pandar_40p_front_base_link']['yaw']}" />
-    <xacro:PandarQT name="pandar_qt_front" parent="front_unit_base_link"
-      x="${calibration['front_unit_base_link2pandar_qt_front_base_link']['x']}"
-      y="${calibration['front_unit_base_link2pandar_qt_front_base_link']['y']}"
-      z="${calibration['front_unit_base_link2pandar_qt_front_base_link']['z']}"
-      roll="${calibration['front_unit_base_link2pandar_qt_front_base_link']['roll']}"
-      pitch="${calibration['front_unit_base_link2pandar_qt_front_base_link']['pitch']}"
-      yaw="${calibration['front_unit_base_link2pandar_qt_front_base_link']['yaw']}" />
+    <xacro:Pandar40P
+      name="pandar_40p_front"
+      parent="front_unit_base_link"
+      x="${calibration['front_unit_base_link']['pandar_40p_front_base_link']['x']}"
+      y="${calibration['front_unit_base_link']['pandar_40p_front_base_link']['y']}"
+      z="${calibration['front_unit_base_link']['pandar_40p_front_base_link']['z']}"
+      roll="${calibration['front_unit_base_link']['pandar_40p_front_base_link']['roll']}"
+      pitch="${calibration['front_unit_base_link']['pandar_40p_front_base_link']['pitch']}"
+      yaw="${calibration['front_unit_base_link']['pandar_40p_front_base_link']['yaw']}"
+    />
+    <xacro:PandarQT
+      name="pandar_qt_front"
+      parent="front_unit_base_link"
+      x="${calibration['front_unit_base_link']['pandar_qt_front_base_link']['x']}"
+      y="${calibration['front_unit_base_link']['pandar_qt_front_base_link']['y']}"
+      z="${calibration['front_unit_base_link']['pandar_qt_front_base_link']['z']}"
+      roll="${calibration['front_unit_base_link']['pandar_qt_front_base_link']['roll']}"
+      pitch="${calibration['front_unit_base_link']['pandar_qt_front_base_link']['pitch']}"
+      yaw="${calibration['front_unit_base_link']['pandar_qt_front_base_link']['yaw']}"
+    />
   </xacro:macro>
 </robot>

File: aip_x2_description/urdf/rear_unit.xacro (robot description, xacro)
@@ -19,28 +19,40 @@
     <xacro:property name="calibration" value="${load_yaml('$(arg config_dir)/rear_unit_calibration.yaml')}"/>
     <!-- BFS4(R) -->
-    <xacro:monocular_camera_macro name="camera3/camera" parent="rear_unit_base_link"
+    <xacro:monocular_camera_macro
+      name="camera3/camera"
+      parent="rear_unit_base_link"
       namespace=""
-      x="${calibration['rear_unit_base_link2camera3']['x']}"
-      y="${calibration['rear_unit_base_link2camera3']['y']}"
-      z="${calibration['rear_unit_base_link2camera3']['z']}"
-      roll="${calibration['rear_unit_base_link2camera3']['roll']}"
-      pitch="${calibration['rear_unit_base_link2camera3']['pitch']}"
-      yaw="${calibration['rear_unit_base_link2camera3']['yaw']}"
-      fps="30" width="800" height="400" fov="1.3"/>
+      x="${calibration['rear_unit_base_link']['camera3/camera_link']['x']}"
+      y="${calibration['rear_unit_base_link']['camera3/camera_link']['y']}"
+      z="${calibration['rear_unit_base_link']['camera3/camera_link']['z']}"
+      roll="${calibration['rear_unit_base_link']['camera3/camera_link']['roll']}"
+      pitch="${calibration['rear_unit_base_link']['camera3/camera_link']['pitch']}"
+      yaw="${calibration['rear_unit_base_link']['camera3/camera_link']['yaw']}"
+      fps="30"
+      width="800"
+      height="400"
+      fov="1.3"
+    />
     <!-- lidar -->
-    <xacro:Pandar40P name="pandar_40p_rear" parent="rear_unit_base_link"
-      x="${calibration['rear_unit_base_link2pandar_40p_rear_base_link']['x']}"
-      y="${calibration['rear_unit_base_link2pandar_40p_rear_base_link']['y']}"
-      z="${calibration['rear_unit_base_link2pandar_40p_rear_base_link']['z']}"
-      roll="${calibration['rear_unit_base_link2pandar_40p_rear_base_link']['roll']}"
-      pitch="${calibration['rear_unit_base_link2pandar_40p_rear_base_link']['pitch']}"
-      yaw="${calibration['rear_unit_base_link2pandar_40p_rear_base_link']['yaw']}" />
-    <xacro:PandarQT name="pandar_qt_rear" parent="rear_unit_base_link"
-      x="${calibration['rear_unit_base_link2pandar_qt_rear_base_link']['x']}"
-      y="${calibration['rear_unit_base_link2pandar_qt_rear_base_link']['y']}"
-      z="${calibration['rear_unit_base_link2pandar_qt_rear_base_link']['z']}"
-      roll="${calibration['rear_unit_base_link2pandar_qt_rear_base_link']['roll']}"
-      pitch="${calibration['rear_unit_base_link2pandar_qt_rear_base_link']['pitch']}"
-      yaw="${calibration['rear_unit_base_link2pandar_qt_rear_base_link']['yaw']}" />
-    </xacro:macro>
+    <xacro:Pandar40P
+      name="pandar_40p_rear"
+      parent="rear_unit_base_link"
+      x="${calibration['rear_unit_base_link']['pandar_40p_rear_base_link']['x']}"
+      y="${calibration['rear_unit_base_link']['pandar_40p_rear_base_link']['y']}"
+      z="${calibration['rear_unit_base_link']['pandar_40p_rear_base_link']['z']}"
+      roll="${calibration['rear_unit_base_link']['pandar_40p_rear_base_link']['roll']}"
+      pitch="${calibration['rear_unit_base_link']['pandar_40p_rear_base_link']['pitch']}"
+      yaw="${calibration['rear_unit_base_link']['pandar_40p_rear_base_link']['yaw']}"
+    />
+    <xacro:PandarQT
+      name="pandar_qt_rear"
+      parent="rear_unit_base_link"
+      x="${calibration['rear_unit_base_link']['pandar_qt_rear_base_link']['x']}"
+      y="${calibration['rear_unit_base_link']['pandar_qt_rear_base_link']['y']}"
+      z="${calibration['rear_unit_base_link']['pandar_qt_rear_base_link']['z']}"
+      roll="${calibration['rear_unit_base_link']['pandar_qt_rear_base_link']['roll']}"
+      pitch="${calibration['rear_unit_base_link']['pandar_qt_rear_base_link']['pitch']}"
+      yaw="${calibration['rear_unit_base_link']['pandar_qt_rear_base_link']['yaw']}"
+    />
+  </xacro:macro>
 </robot>

File: aip_x2_description/urdf/sensors.xacro (robot description, xacro)
@@ -1,15 +1,38 @@
 <?xml version="1.0"?>
-<robot name="vehicle"
-  xmlns:xacro="http://ros.org/wiki/xacro">
+<robot name="vehicle" xmlns:xacro="http://ros.org/wiki/xacro">
   <xacro:arg name="config_dir" default="$(find aip_x2_description)/config"/>
   <xacro:property name="calibration" value="${load_yaml('$(arg config_dir)/sensors_calibration.yaml')}"/>
   <!-- top unit -->
   <xacro:include filename="top_unit.xacro"/>
-  <xacro:top_unit_macro parent="base_link" x="${calibration['base_link2top_unit_base_link']['x']}" y="${calibration['base_link2top_unit_base_link']['y']}" z="${calibration['base_link2top_unit_base_link']['z']}" roll="${calibration['base_link2top_unit_base_link']['roll']}" pitch="${calibration['base_link2top_unit_base_link']['pitch']}" yaw="${calibration['base_link2top_unit_base_link']['yaw']}" />
+  <xacro:top_unit_macro
+    parent="base_link"
+    x="${calibration['base_link']['top_unit_base_link']['x']}"
+    y="${calibration['base_link']['top_unit_base_link']['y']}"
+    z="${calibration['base_link']['top_unit_base_link']['z']}"
+    roll="${calibration['base_link']['top_unit_base_link']['roll']}"
+    pitch="${calibration['base_link']['top_unit_base_link']['pitch']}"
+    yaw="${calibration['base_link']['top_unit_base_link']['yaw']}"
+  />
   <!-- front unit -->
   <xacro:include filename="front_unit.xacro"/>
-  <xacro:front_unit_macro parent="base_link" x="${calibration['base_link2front_unit_base_link']['x']}" y="${calibration['base_link2front_unit_base_link']['y']}" z="${calibration['base_link2front_unit_base_link']['z']}" roll="${calibration['base_link2front_unit_base_link']['roll']}" pitch="${calibration['base_link2front_unit_base_link']['pitch']}" yaw="${calibration['base_link2front_unit_base_link']['yaw']}" />
+  <xacro:front_unit_macro
+    parent="base_link"
+    x="${calibration['base_link']['front_unit_base_link']['x']}"
+    y="${calibration['base_link']['front_unit_base_link']['y']}"
+    z="${calibration['base_link']['front_unit_base_link']['z']}"
+    roll="${calibration['base_link']['front_unit_base_link']['roll']}"
+    pitch="${calibration['base_link']['front_unit_base_link']['pitch']}"
+    yaw="${calibration['base_link']['front_unit_base_link']['yaw']}"
+  />
   <!-- rear unit -->
   <xacro:include filename="rear_unit.xacro"/>
-  <xacro:rear_unit_macro parent="base_link" x="${calibration['base_link2rear_unit_base_link']['x']}" y="${calibration['base_link2rear_unit_base_link']['y']}" z="${calibration['base_link2rear_unit_base_link']['z']}" roll="${calibration['base_link2rear_unit_base_link']['roll']}" pitch="${calibration['base_link2rear_unit_base_link']['pitch']}" yaw="${calibration['base_link2rear_unit_base_link']['yaw']}" />
+  <xacro:rear_unit_macro
+    parent="base_link"
+    x="${calibration['base_link']['rear_unit_base_link']['x']}"
+    y="${calibration['base_link']['rear_unit_base_link']['y']}"
+    z="${calibration['base_link']['rear_unit_base_link']['z']}"
+    roll="${calibration['base_link']['rear_unit_base_link']['roll']}"
+    pitch="${calibration['base_link']['rear_unit_base_link']['pitch']}"
+    yaw="${calibration['base_link']['rear_unit_base_link']['yaw']}"
+  />
 </robot>
