Commit message: Modify sensor config (#4)
* Update x1 sensor config files

Signed-off-by: wep21 <border_goldenmarket@yahoo.co.jp>

* Update xx1 sensor config files

Signed-off-by: wep21 <border_goldenmarket@yahoo.co.jp>

* Update x2 sensor config files

Signed-off-by: wep21 <border_goldenmarket@yahoo.co.jp>

* Run pre-commit

Signed-off-by: wep21 <border_goldenmarket@yahoo.co.jp>

* Add prettier-xacro to pre-commit (#6)

Signed-off-by: Kenji Miyake <kenji.miyake@tier4.jp>

* Run pre-commit

Signed-off-by: wep21 <border_goldenmarket@yahoo.co.jp>

* Update README.md

Signed-off-by: wep21 <border_goldenmarket@yahoo.co.jp>

* Fix for pre-commit

Signed-off-by: Kenji Miyake <kenji.miyake@tier4.jp>

* Cosmetic change

Signed-off-by: wep21 <border_goldenmarket@yahoo.co.jp>

* Add _link

Signed-off-by: wep21 <border_goldenmarket@yahoo.co.jp>

* Fix missing link

Co-authored-by: Kenji Miyake <31987104+kenji-miyake@users.noreply.github.com>
Co-authored-by: Kenji Miyake <kenji.miyake@tier4.jp>

File: aip_x2_description/urdf/top_unit.xacro (robot description, xacro)
@@ -21,48 +21,144 @@
     <!-- lidar -->
     <!-- left -->
-    <xacro:Pandar40P name="pandar_40p_left" parent="top_unit_base_link"
-      x="${calibration['top_unit_base_link2pandar_40p_left_base_link']['x']}"
-      y="${calibration['top_unit_base_link2pandar_40p_left_base_link']['y']}"
-      z="${calibration['top_unit_base_link2pandar_40p_left_base_link']['z']}"
-      roll="${calibration['top_unit_base_link2pandar_40p_left_base_link']['roll']}"
-      pitch="${calibration['top_unit_base_link2pandar_40p_left_base_link']['pitch']}"
-      yaw="${calibration['top_unit_base_link2pandar_40p_left_base_link']['yaw']}" />
-    <xacro:PandarQT name="pandar_qt_left" parent="top_unit_base_link"
-      x="${calibration['top_unit_base_link2pandar_qt_left_base_link']['x']}"
-      y="${calibration['top_unit_base_link2pandar_qt_left_base_link']['y']}"
-      z="${calibration['top_unit_base_link2pandar_qt_left_base_link']['z']}"
-      roll="${calibration['top_unit_base_link2pandar_qt_left_base_link']['roll']}"
-      pitch="${calibration['top_unit_base_link2pandar_qt_left_base_link']['pitch']}"
-      yaw="${calibration['top_unit_base_link2pandar_qt_left_base_link']['yaw']}" />
+    <xacro:Pandar40P
+      name="pandar_40p_left"
+      parent="top_unit_base_link"
+      x="${calibration['top_unit_base_link']['pandar_40p_left_base_link']['x']}"
+      y="${calibration['top_unit_base_link']['pandar_40p_left_base_link']['y']}"
+      z="${calibration['top_unit_base_link']['pandar_40p_left_base_link']['z']}"
+      roll="${calibration['top_unit_base_link']['pandar_40p_left_base_link']['roll']}"
+      pitch="${calibration['top_unit_base_link']['pandar_40p_left_base_link']['pitch']}"
+      yaw="${calibration['top_unit_base_link']['pandar_40p_left_base_link']['yaw']}"
+    />
+    <xacro:PandarQT
+      name="pandar_qt_left"
+      parent="top_unit_base_link"
+      x="${calibration['top_unit_base_link']['pandar_qt_left_base_link']['x']}"
+      y="${calibration['top_unit_base_link']['pandar_qt_left_base_link']['y']}"
+      z="${calibration['top_unit_base_link']['pandar_qt_left_base_link']['z']}"
+      roll="${calibration['top_unit_base_link']['pandar_qt_left_base_link']['roll']}"
+      pitch="${calibration['top_unit_base_link']['pandar_qt_left_base_link']['pitch']}"
+      yaw="${calibration['top_unit_base_link']['pandar_qt_left_base_link']['yaw']}"
+    />
     <!-- right -->
-    <xacro:Pandar40P name="pandar_40p_right" parent="top_unit_base_link"
-      x="${calibration['top_unit_base_link2pandar_40p_right_base_link']['x']}"
-      y="${calibration['top_unit_base_link2pandar_40p_right_base_link']['y']}"
-      z="${calibration['top_unit_base_link2pandar_40p_right_base_link']['z']}"
-      roll="${calibration['top_unit_base_link2pandar_40p_right_base_link']['roll']}"
-      pitch="${calibration['top_unit_base_link2pandar_40p_right_base_link']['pitch']}"
-      yaw="${calibration['top_unit_base_link2pandar_40p_right_base_link']['yaw']}" />
-    <xacro:PandarQT name="pandar_qt_right" parent="top_unit_base_link"
-      x="${calibration['top_unit_base_link2pandar_qt_right_base_link']['x']}"
-      y="${calibration['top_unit_base_link2pandar_qt_right_base_link']['y']}"
-      z="${calibration['top_unit_base_link2pandar_qt_right_base_link']['z']}"
-      roll="${calibration['top_unit_base_link2pandar_qt_right_base_link']['roll']}"
-      pitch="${calibration['top_unit_base_link2pandar_qt_right_base_link']['pitch']}"
-      yaw="${calibration['top_unit_base_link2pandar_qt_right_base_link']['yaw']}" />
+    <xacro:Pandar40P
+      name="pandar_40p_right"
+      parent="top_unit_base_link"
+      x="${calibration['top_unit_base_link']['pandar_40p_right_base_link']['x']}"
+      y="${calibration['top_unit_base_link']['pandar_40p_right_base_link']['y']}"
+      z="${calibration['top_unit_base_link']['pandar_40p_right_base_link']['z']}"
+      roll="${calibration['top_unit_base_link']['pandar_40p_right_base_link']['roll']}"
+      pitch="${calibration['top_unit_base_link']['pandar_40p_right_base_link']['pitch']}"
+      yaw="${calibration['top_unit_base_link']['pandar_40p_right_base_link']['yaw']}"
+    />
+    <xacro:PandarQT
+      name="pandar_qt_right"
+      parent="top_unit_base_link"
+      x="${calibration['top_unit_base_link']['pandar_qt_right_base_link']['x']}"
+      y="${calibration['top_unit_base_link']['pandar_qt_right_base_link']['y']}"
+      z="${calibration['top_unit_base_link']['pandar_qt_right_base_link']['z']}"
+      roll="${calibration['top_unit_base_link']['pandar_qt_right_base_link']['roll']}"
+      pitch="${calibration['top_unit_base_link']['pandar_qt_right_base_link']['pitch']}"
+      yaw="${calibration['top_unit_base_link']['pandar_qt_right_base_link']['yaw']}"
+    />
     <!-- camera -->
     <!-- TLR -->
-    <xacro:monocular_camera_macro name="traffic_light_camera/camera" parent="top_unit_base_link" namespace="" x="${calibration['top_unit_base_link2traffic_light_camera']['x']}" y="${calibration['top_unit_base_link2traffic_light_camera']['y']}" z="${calibration['top_unit_base_link2traffic_light_camera']['z']}" roll="${calibration['top_unit_base_link2traffic_light_camera']['roll']}" pitch="${calibration['top_unit_base_link2traffic_light_camera']['pitch']}" yaw="${calibration['top_unit_base_link2traffic_light_camera']['yaw']}" fps="30" width="800" height="400" fov="1.3"/>
+    <xacro:monocular_camera_macro
+      name="traffic_light_camera/camera"
+      parent="top_unit_base_link"
+      namespace=""
+      x="${calibration['top_unit_base_link']['traffic_light_camera_link']['x']}"
+      y="${calibration['top_unit_base_link']['traffic_light_camera_link']['y']}"
+      z="${calibration['top_unit_base_link']['traffic_light_camera_link']['z']}"
+      roll="${calibration['top_unit_base_link']['traffic_light_camera_link']['roll']}"
+      pitch="${calibration['top_unit_base_link']['traffic_light_camera_link']['pitch']}"
+      yaw="${calibration['top_unit_base_link']['traffic_light_camera_link']['yaw']}"
+      fps="30"
+      width="800"
+      height="400"
+      fov="1.3"
+    />
     <!-- BFS1(F) -->
-    <xacro:monocular_camera_macro name="camera0/camera" parent="top_unit_base_link" namespace="" x="${calibration['top_unit_base_link2camera0']['x']}" y="${calibration['top_unit_base_link2camera0']['y']}" z="${calibration['top_unit_base_link2camera0']['z']}" roll="${calibration['top_unit_base_link2camera0']['roll']}" pitch="${calibration['top_unit_base_link2camera0']['pitch']}" yaw="${calibration['top_unit_base_link2camera0']['yaw']}" fps="30" width="800" height="400" fov="1.3"/>
+    <xacro:monocular_camera_macro
+      name="camera0/camera"
+      parent="top_unit_base_link"
+      namespace=""
+      x="${calibration['top_unit_base_link']['camera0/camera_link']['x']}"
+      y="${calibration['top_unit_base_link']['camera0/camera_link']['y']}"
+      z="${calibration['top_unit_base_link']['camera0/camera_link']['z']}"
+      roll="${calibration['top_unit_base_link']['camera0/camera_link']['roll']}"
+      pitch="${calibration['top_unit_base_link']['camera0/camera_link']['pitch']}"
+      yaw="${calibration['top_unit_base_link']['camera0/camera_link']['yaw']}"
+      fps="30"
+      width="800"
+      height="400"
+      fov="1.3"
+    />
     <!-- BFS2(RF) -->
-    <xacro:monocular_camera_macro name="camera1/camera" parent="top_unit_base_link" namespace="" x="${calibration['top_unit_base_link2camera1']['x']}" y="${calibration['top_unit_base_link2camera1']['y']}" z="${calibration['top_unit_base_link2camera1']['z']}" roll="${calibration['top_unit_base_link2camera1']['roll']}" pitch="${calibration['top_unit_base_link2camera1']['pitch']}" yaw="${calibration['top_unit_base_link2camera1']['yaw']}" fps="30" width="800" height="400" fov="1.3"/>
+    <xacro:monocular_camera_macro
+      name="camera1/camera"
+      parent="top_unit_base_link"
+      namespace=""
+      x="${calibration['top_unit_base_link']['camera1/camera_link']['x']}"
+      y="${calibration['top_unit_base_link']['camera1/camera_link']['y']}"
+      z="${calibration['top_unit_base_link']['camera1/camera_link']['z']}"
+      roll="${calibration['top_unit_base_link']['camera1/camera_link']['roll']}"
+      pitch="${calibration['top_unit_base_link']['camera1/camera_link']['pitch']}"
+      yaw="${calibration['top_unit_base_link']['camera1/camera_link']['yaw']}"
+      fps="30"
+      width="800"
+      height="400"
+      fov="1.3"
+    />
     <!-- BFS3(RR) -->
-    <xacro:monocular_camera_macro name="camera2/camera" parent="top_unit_base_link" namespace="" x="${calibration['top_unit_base_link2camera2']['x']}" y="${calibration['top_unit_base_link2camera2']['y']}" z="${calibration['top_unit_base_link2camera2']['z']}" roll="${calibration['top_unit_base_link2camera2']['roll']}" pitch="${calibration['top_unit_base_link2camera2']['pitch']}" yaw="${calibration['top_unit_base_link2camera2']['yaw']}" fps="30" width="800" height="400" fov="1.3"/>
+    <xacro:monocular_camera_macro
+      name="camera2/camera"
+      parent="top_unit_base_link"
+      namespace=""
+      x="${calibration['top_unit_base_link']['camera2/camera_link']['x']}"
+      y="${calibration['top_unit_base_link']['camera2/camera_link']['y']}"
+      z="${calibration['top_unit_base_link']['camera2/camera_link']['z']}"
+      roll="${calibration['top_unit_base_link']['camera2/camera_link']['roll']}"
+      pitch="${calibration['top_unit_base_link']['camera2/camera_link']['pitch']}"
+      yaw="${calibration['top_unit_base_link']['camera2/camera_link']['yaw']}"
+      fps="30"
+      width="800"
+      height="400"
+      fov="1.3"
+    />
     <!-- BFS4(R) -->
     <!-- embedded! -->
     <!-- BFS5(LR) -->
-    <xacro:monocular_camera_macro name="camera4/camera" parent="top_unit_base_link" namespace="" x="${calibration['top_unit_base_link2camera4']['x']}" y="${calibration['top_unit_base_link2camera4']['y']}" z="${calibration['top_unit_base_link2camera4']['z']}" roll="${calibration['top_unit_base_link2camera4']['roll']}" pitch="${calibration['top_unit_base_link2camera4']['pitch']}" yaw="${calibration['top_unit_base_link2camera4']['yaw']}" fps="30" width="800" height="400" fov="1.3"/>
+    <xacro:monocular_camera_macro
+      name="camera4/camera"
+      parent="top_unit_base_link"
+      namespace=""
+      x="${calibration['top_unit_base_link']['camera4/camera_link']['x']}"
+      y="${calibration['top_unit_base_link']['camera4/camera_link']['y']}"
+      z="${calibration['top_unit_base_link']['camera4/camera_link']['z']}"
+      roll="${calibration['top_unit_base_link']['camera4/camera_link']['roll']}"
+      pitch="${calibration['top_unit_base_link']['camera4/camera_link']['pitch']}"
+      yaw="${calibration['top_unit_base_link']['camera4/camera_link']['yaw']}"
+      fps="30"
+      width="800"
+      height="400"
+      fov="1.3"
+    />
     <!-- BFS6(LR) -->
-    <xacro:monocular_camera_macro name="camera5/camera" parent="top_unit_base_link" namespace="" x="${calibration['top_unit_base_link2camera5']['x']}" y="${calibration['top_unit_base_link2camera5']['y']}" z="${calibration['top_unit_base_link2camera5']['z']}" roll="${calibration['top_unit_base_link2camera5']['roll']}" pitch="${calibration['top_unit_base_link2camera5']['pitch']}" yaw="${calibration['top_unit_base_link2camera5']['yaw']}" fps="30" width="800" height="400" fov="1.3"/>
+    <xacro:monocular_camera_macro
+      name="camera5/camera"
+      parent="top_unit_base_link"
+      namespace=""
+      x="${calibration['top_unit_base_link']['camera5/camera_link']['x']}"
+      y="${calibration['top_unit_base_link']['camera5/camera_link']['y']}"
+      z="${calibration['top_unit_base_link']['camera5/camera_link']['z']}"
+      roll="${calibration['top_unit_base_link']['camera5/camera_link']['roll']}"
+      pitch="${calibration['top_unit_base_link']['camera5/camera_link']['pitch']}"
+      yaw="${calibration['top_unit_base_link']['camera5/camera_link']['yaw']}"
+      fps="30"
+      width="800"
+      height="400"
+      fov="1.3"
+    />
     <!-- gnss -->
     <!-- left -->
@@ -71,11 +167,12 @@
       parent="top_unit_base_link"
       namespace=""
-      x="${calibration['top_unit_base_link2gnss_right']['x']}"
-      y="${calibration['top_unit_base_link2gnss_right']['y']}"
-      z="${calibration['top_unit_base_link2gnss_right']['z']}"
-      roll="${calibration['top_unit_base_link2gnss_right']['roll']}"
-      pitch="${calibration['top_unit_base_link2gnss_right']['pitch']}"
-      yaw="${calibration['top_unit_base_link2gnss_right']['yaw']}"
-      fps="100" />
+      x="${calibration['top_unit_base_link']['gnss_right_link']['x']}"
+      y="${calibration['top_unit_base_link']['gnss_right_link']['y']}"
+      z="${calibration['top_unit_base_link']['gnss_right_link']['z']}"
+      roll="${calibration['top_unit_base_link']['gnss_right_link']['roll']}"
+      pitch="${calibration['top_unit_base_link']['gnss_right_link']['pitch']}"
+      yaw="${calibration['top_unit_base_link']['gnss_right_link']['yaw']}"
+      fps="100"
+    />
     <!-- right -->
     <xacro:imu_macro
@@ -83,11 +180,12 @@
       parent="top_unit_base_link"
       namespace=""
-      x="${calibration['top_unit_base_link2gnss_left']['x']}"
-      y="${calibration['top_unit_base_link2gnss_left']['y']}"
-      z="${calibration['top_unit_base_link2gnss_left']['z']}"
-      roll="${calibration['top_unit_base_link2gnss_left']['roll']}"
-      pitch="${calibration['top_unit_base_link2gnss_left']['pitch']}"
-      yaw="${calibration['top_unit_base_link2gnss_left']['yaw']}"
-      fps="100" />
+      x="${calibration['top_unit_base_link']['gnss_left_link']['x']}"
+      y="${calibration['top_unit_base_link']['gnss_left_link']['y']}"
+      z="${calibration['top_unit_base_link']['gnss_left_link']['z']}"
+      roll="${calibration['top_unit_base_link']['gnss_left_link']['roll']}"
+      pitch="${calibration['top_unit_base_link']['gnss_left_link']['pitch']}"
+      yaw="${calibration['top_unit_base_link']['gnss_left_link']['yaw']}"
+      fps="100"
+    />
     <!-- imu -->
     <xacro:imu_macro
@@ -95,11 +193,12 @@
       parent="top_unit_base_link"
       namespace=""
-      x="${calibration['top_unit_base_link2imu_tamagawa']['x']}"
-      y="${calibration['top_unit_base_link2imu_tamagawa']['y']}"
-      z="${calibration['top_unit_base_link2imu_tamagawa']['z']}"
-      roll="${calibration['top_unit_base_link2imu_tamagawa']['roll']}"
-      pitch="${calibration['top_unit_base_link2imu_tamagawa']['pitch']}"
-      yaw="${calibration['top_unit_base_link2imu_tamagawa']['yaw']}"
-      fps="100" />
+      x="${calibration['top_unit_base_link']['tamagawa/imu_link']['x']}"
+      y="${calibration['top_unit_base_link']['tamagawa/imu_link']['y']}"
+      z="${calibration['top_unit_base_link']['tamagawa/imu_link']['z']}"
+      roll="${calibration['top_unit_base_link']['tamagawa/imu_link']['roll']}"
+      pitch="${calibration['top_unit_base_link']['tamagawa/imu_link']['pitch']}"
+      yaw="${calibration['top_unit_base_link']['tamagawa/imu_link']['yaw']}"
+      fps="100"
+    />
   </xacro:macro>
 </robot>

Commit message: fix(aip_x*_description): fix xacro deprecated usage
Signed-off-by: Takayuki Murooka <takayuki5168@gmail.com>

File: aip_x1_description/urdf/sensor_kit.xacro (robot description, xacro)
@@ -15,5 +15,5 @@
     </link>
     <!-- sensor -->
-    <xacro:property name="calibration" value="${load_yaml('$(arg config_dir)/sensor_kit_calibration.yaml')}"/>
+    <xacro:property name="calibration" value="${xacro.load_yaml('$(arg config_dir)/sensor_kit_calibration.yaml')}"/>
     <!-- lidar -->
     <xacro:VLP-16

File: aip_x2_description/urdf/front_unit.xacro (robot description, xacro)
@@ -17,5 +17,5 @@
     </link>
     <!-- sensor -->
-    <xacro:property name="calibration" value="${load_yaml('$(arg config_dir)/front_unit_calibration.yaml')}"/>
+    <xacro:property name="calibration" value="${xacro.load_yaml('$(arg config_dir)/front_unit_calibration.yaml')}"/>
     <!-- BFS7(LR) -->
     <xacro:monocular_camera_macro

File: aip_x2_description/urdf/rear_unit.xacro (robot description, xacro)
@@ -17,5 +17,5 @@
     </link>
     <!-- sensor -->
-    <xacro:property name="calibration" value="${load_yaml('$(arg config_dir)/rear_unit_calibration.yaml')}"/>
+    <xacro:property name="calibration" value="${xacro.load_yaml('$(arg config_dir)/rear_unit_calibration.yaml')}"/>
     <!-- BFS4(R) -->
     <xacro:monocular_camera_macro

File: aip_x2_description/urdf/sensors.xacro (robot description, xacro)
@@ -2,5 +2,5 @@
 <robot name="vehicle" xmlns:xacro="http://ros.org/wiki/xacro">
   <xacro:arg name="config_dir" default="$(find aip_x2_description)/config"/>
-  <xacro:property name="calibration" value="${load_yaml('$(arg config_dir)/sensors_calibration.yaml')}"/>
+  <xacro:property name="calibration" value="${xacro.load_yaml('$(arg config_dir)/sensors_calibration.yaml')}"/>
   <!-- top unit -->
   <xacro:include filename="top_unit.xacro"/>

File: aip_x2_description/urdf/top_unit.xacro (robot description, xacro)
@@ -18,5 +18,5 @@
     </link>
     <!-- sensor -->
-    <xacro:property name="calibration" value="${load_yaml('$(arg config_dir)/top_unit_calibration.yaml')}"/>
+    <xacro:property name="calibration" value="${xacro.load_yaml('$(arg config_dir)/top_unit_calibration.yaml')}"/>
     <!-- lidar -->
     <!-- left -->

Commit message: chore: remove aip_x1 and rename aip_x1_1 to aip_x1
Signed-off-by: 1222-takeshi <m.takeshi1995@gmail.com>

File: aip_x1_description/urdf/sensor_kit.xacro (robot description, xacro)
@@ -5,5 +5,5 @@
     <xacro:include filename="$(find imu_description)/urdf/imu.xacro"/>
     <xacro:arg name="gpu" default="false"/>
-    <xacro:arg name="config_dir" default="$(find aip_x1_description)/config"/>
+    <xacro:arg name="config_dir" default="$(find aip_x1_1_description)/config"/>
     <xacro:property name="sensor_kit_base_link" default="sensor_kit_base_link"/>
     <joint name="${sensor_kit_base_link}_joint" type="fixed">
@@ -16,5 +16,5 @@
     </link>
     <!-- sensor -->
-    <xacro:property name="calibration" value="${xacro.load_yaml('$(arg config_dir)/sensor_kit_calibration.yaml')}"/>
+    <xacro:property name="calibration" value="${load_yaml('$(arg config_dir)/sensor_kit_calibration.yaml')}"/>
     <!-- lidar -->
     <xacro:VLP-16
@@ -35,34 +35,14 @@
       />
     </xacro:VLP-16>
-    <xacro:include filename="$(find livox_description)/urdf/livox_horizon.xacro"/>
-    <xacro:livox_horizon_macro
-      name="livox_front_left"
+    <xacro:include filename="$(find pandar_description)/urdf/pandar_xt32.xacro"/>
+    <xacro:PandarXT-32
+      name="pandar_xt32_front_center"
       parent="sensor_kit_base_link"
-      x="${calibration['sensor_kit_base_link']['livox_front_left_base_link']['x']}"
-      y="${calibration['sensor_kit_base_link']['livox_front_left_base_link']['y']}"
-      z="${calibration['sensor_kit_base_link']['livox_front_left_base_link']['z']}"
-      roll="${calibration['sensor_kit_base_link']['livox_front_left_base_link']['roll']}"
-      pitch="${calibration['sensor_kit_base_link']['livox_front_left_base_link']['pitch']}"
-      yaw="${calibration['sensor_kit_base_link']['livox_front_left_base_link']['yaw']}"
-    />
-    <xacro:livox_horizon_macro
-      name="livox_front_center"
-      parent="sensor_kit_base_link"
-      x="${calibration['sensor_kit_base_link']['livox_front_center_base_link']['x']}"
-      y="${calibration['sensor_kit_base_link']['livox_front_center_base_link']['y']}"
-      z="${calibration['sensor_kit_base_link']['livox_front_center_base_link']['z']}"
-      roll="${calibration['sensor_kit_base_link']['livox_front_center_base_link']['roll']}"
-      pitch="${calibration['sensor_kit_base_link']['livox_front_center_base_link']['pitch']}"
-      yaw="${calibration['sensor_kit_base_link']['livox_front_center_base_link']['yaw']}"
-    />
-    <xacro:livox_horizon_macro
-      name="livox_front_right"
-      parent="sensor_kit_base_link"
-      x="${calibration['sensor_kit_base_link']['livox_front_right_base_link']['x']}"
-      y="${calibration['sensor_kit_base_link']['livox_front_right_base_link']['y']}"
-      z="${calibration['sensor_kit_base_link']['livox_front_right_base_link']['z']}"
-      roll="${calibration['sensor_kit_base_link']['livox_front_right_base_link']['roll']}"
-      pitch="${calibration['sensor_kit_base_link']['livox_front_right_base_link']['pitch']}"
-      yaw="${calibration['sensor_kit_base_link']['livox_front_right_base_link']['yaw']}"
+      x="${calibration['sensor_kit_base_link']['pandar_xt32_front_center_base_link']['x']}"
+      y="${calibration['sensor_kit_base_link']['pandar_xt32_front_center_base_link']['y']}"
+      z="${calibration['sensor_kit_base_link']['pandar_xt32_front_center_base_link']['z']}"
+      roll="${calibration['sensor_kit_base_link']['pandar_xt32_front_center_base_link']['roll']}"
+      pitch="${calibration['sensor_kit_base_link']['pandar_xt32_front_center_base_link']['pitch']}"
+      yaw="${calibration['sensor_kit_base_link']['pandar_xt32_front_center_base_link']['yaw']}"
     />
     <!-- gnss -->

Commit message: chore: remove unused file and fix bug
Signed-off-by: 1222-takeshi <m.takeshi1995@gmail.com>

File: aip_x1_description/urdf/sensor_kit.xacro (robot description, xacro)
@@ -16,5 +16,5 @@
     </link>
     <!-- sensor -->
-    <xacro:property name="calibration" value="${load_yaml('$(arg config_dir)/sensor_kit_calibration.yaml')}"/>
+    <xacro:property name="calibration" value="${xacro.load_yaml('$(arg config_dir)/sensor_kit_calibration.yaml')}"/>
     <!-- lidar -->
     <xacro:VLP-16
