Commit message: change: front lidar

File: aip_x1_description/urdf/sensor_kit.xacro (robot description, xacro)
@@ -35,15 +35,22 @@
       />
     </xacro:VLP-16>
-    <xacro:include filename="$(find pandar_description)/urdf/pandar_xt32.xacro"/>
-    <xacro:PandarXT-32
-      name="pandar_xt32_front_center"
+    <xacro:include filename="$(find velodyne_description)/urdf/VLP-32C.urdf.xacro"/>
+    <xacro:VLP-32C
       parent="sensor_kit_base_link"
-      x="${calibration['sensor_kit_base_link']['pandar_xt32_front_center_base_link']['x']}"
-      y="${calibration['sensor_kit_base_link']['pandar_xt32_front_center_base_link']['y']}"
-      z="${calibration['sensor_kit_base_link']['pandar_xt32_front_center_base_link']['z']}"
-      roll="${calibration['sensor_kit_base_link']['pandar_xt32_front_center_base_link']['roll']}"
-      pitch="${calibration['sensor_kit_base_link']['pandar_xt32_front_center_base_link']['pitch']}"
-      yaw="${calibration['sensor_kit_base_link']['pandar_xt32_front_center_base_link']['yaw']}"
-    />
+      name="velodyne_front_center"
+      topic="/points_raw"
+      hz="10"
+      samples="220"
+      gpu="$(arg gpu)"
+    >
+      <origin
+        xyz="${calibration['sensor_kit_base_link']['velodyne_front_center_base_link']['x']}
+             ${calibration['sensor_kit_base_link']['velodyne_front_center_base_link']['y']}
+             ${calibration['sensor_kit_base_link']['velodyne_front_center_base_link']['z']}"
+        rpy="${calibration['sensor_kit_base_link']['velodyne_front_center_base_link']['roll']}
+             ${calibration['sensor_kit_base_link']['velodyne_front_center_base_link']['pitch']}
+             ${calibration['sensor_kit_base_link']['velodyne_front_center_base_link']['yaw']}"
+      />
+    </xacro:VLP-32C>
     <!-- gnss -->
     <xacro:imu_macro
