Commit message: update for xx1 gen2
Signed-off-by: Yukihiro Saito <yukky.saito@gmail.com>

File: aip_xx1_description/urdf/sensor_kit.xacro (robot description, xacro)
@@ -2,7 +2,6 @@
 <robot xmlns:xacro="http://ros.org/wiki/xacro">
   <xacro:macro name="sensor_kit_macro" params="parent x y z roll pitch yaw">
-    <xacro:include filename="$(find velodyne_description)/urdf/HDL-32E.urdf.xacro"/>
+    <xacro:include filename="$(find pandar_description)/urdf/pandar_xt32.xacro"/>
     <xacro:include filename="$(find velodyne_description)/urdf/VLP-16.urdf.xacro"/>
-    <xacro:include filename="$(find vls_description)/urdf/VLS-128.urdf.xacro"/>
     <xacro:include filename="$(find camera_description)/urdf/monocular_camera.xacro"/>
     <xacro:include filename="$(find imu_description)/urdf/imu.xacro"/>
@@ -22,55 +21,34 @@
     <xacro:property name="calibration" value="${xacro.load_yaml('$(arg config_dir)/sensor_kit_calibration.yaml')}"/>
     <!-- lidar -->
-    <xacro:VLS-128
-      parent="sensor_kit_base_link"
-      name="velodyne_top"
-      topic="/points_raw"
-      hz="10"
-      samples="220"
-      gpu="$(arg gpu)"
-    >
-      <origin
-        xyz="${calibration['sensor_kit_base_link']['velodyne_top_base_link']['x']}
-             ${calibration['sensor_kit_base_link']['velodyne_top_base_link']['y']}
-             ${calibration['sensor_kit_base_link']['velodyne_top_base_link']['z']}"
-        rpy="${calibration['sensor_kit_base_link']['velodyne_top_base_link']['roll']}
-             ${calibration['sensor_kit_base_link']['velodyne_top_base_link']['pitch']}
-             ${calibration['sensor_kit_base_link']['velodyne_top_base_link']['yaw']}"
-      />
-    </xacro:VLS-128>
-    <xacro:VLP-16
-      parent="sensor_kit_base_link"
-      name="velodyne_left"
-      topic="/points_raw"
-      hz="10"
-      samples="220"
-      gpu="$(arg gpu)"
-    >
-      <origin
-        xyz="${calibration['sensor_kit_base_link']['velodyne_left_base_link']['x']}
-             ${calibration['sensor_kit_base_link']['velodyne_left_base_link']['y']}
-             ${calibration['sensor_kit_base_link']['velodyne_left_base_link']['z']}"
-        rpy="${calibration['sensor_kit_base_link']['velodyne_left_base_link']['roll']}
-             ${calibration['sensor_kit_base_link']['velodyne_left_base_link']['pitch']}
-             ${calibration['sensor_kit_base_link']['velodyne_left_base_link']['yaw']}"
-      />
-    </xacro:VLP-16>
-    <xacro:VLP-16
-      parent="sensor_kit_base_link"
-      name="velodyne_right"
-      topic="/points_raw"
-      hz="10"
-      samples="220"
-      gpu="$(arg gpu)"
-    >
-      <origin
-        xyz="${calibration['sensor_kit_base_link']['velodyne_right_base_link']['x']}
-             ${calibration['sensor_kit_base_link']['velodyne_right_base_link']['y']}
-             ${calibration['sensor_kit_base_link']['velodyne_right_base_link']['z']}"
-        rpy="${calibration['sensor_kit_base_link']['velodyne_right_base_link']['roll']}
-             ${calibration['sensor_kit_base_link']['velodyne_right_base_link']['pitch']}
-             ${calibration['sensor_kit_base_link']['velodyne_right_base_link']['yaw']}"
-      />
-    </xacro:VLP-16>
+    <xacro:PandarXT-32
+      name="hesai_top"
+      parent="sensor_kit_base_link"
+      x="${calibration['sensor_kit_base_link']['hesai_top_base_link']['x']}"
+      y="${calibration['sensor_kit_base_link']['hesai_top_base_link']['y']}"
+      z="${calibration['sensor_kit_base_link']['hesai_top_base_link']['z']}"
+      roll="${calibration['sensor_kit_base_link']['hesai_top_base_link']['roll']}"
+      pitch="${calibration['sensor_kit_base_link']['hesai_top_base_link']['pitch']}"
+      yaw="${calibration['sensor_kit_base_link']['hesai_top_base_link']['yaw']}"
+    />
+    <xacro:PandarXT-32
+      name="hesai_right"
+      parent="sensor_kit_base_link"
+      x="${calibration['sensor_kit_base_link']['hesai_right_base_link']['x']}"
+      y="${calibration['sensor_kit_base_link']['hesai_right_base_link']['y']}"
+      z="${calibration['sensor_kit_base_link']['hesai_right_base_link']['z']}"
+      roll="${calibration['sensor_kit_base_link']['hesai_right_base_link']['roll']}"
+      pitch="${calibration['sensor_kit_base_link']['hesai_right_base_link']['pitch']}"
+      yaw="${calibration['sensor_kit_base_link']['hesai_right_base_link']['yaw']}"
+    />
+    <xacro:PandarXT-32
+      name="hesai_left"
+      parent="sensor_kit_base_link"
+      x="${calibration['sensor_kit_base_link']['hesai_left_base_link']['x']}"
+      y="${calibration['sensor_kit_base_link']['hesai_left_base_link']['y']}"
+      z="${calibration['sensor_kit_base_link']['hesai_left_base_link']['z']}"
+      roll="${calibration['sensor_kit_base_link']['hesai_left_base_link']['roll']}"
+      pitch="${calibration['sensor_kit_base_link']['hesai_left_base_link']['pitch']}"
+      yaw="${calibration['sensor_kit_base_link']['hesai_left_base_link']['yaw']}"
+    />
     <!-- camera -->
     <xacro:monocular_camera_macro
@@ -189,4 +167,49 @@
       pitch="${calibration['sensor_kit_base_link']['camera7/camera_link']['pitch']}"
       yaw="${calibration['sensor_kit_base_link']['camera7/camera_link']['yaw']}"
+      fps="30"
+      width="800"
+      height="400"
+      fov="1.3"
+    />
+    <xacro:monocular_camera_macro
+      name="camera8/camera"
+      parent="sensor_kit_base_link"
+      namespace=""
+      x="${calibration['sensor_kit_base_link']['camera8/camera_link']['x']}"
+      y="${calibration['sensor_kit_base_link']['camera8/camera_link']['y']}"
+      z="${calibration['sensor_kit_base_link']['camera8/camera_link']['z']}"
+      roll="${calibration['sensor_kit_base_link']['camera8/camera_link']['roll']}"
+      pitch="${calibration['sensor_kit_base_link']['camera8/camera_link']['pitch']}"
+      yaw="${calibration['sensor_kit_base_link']['camera8/camera_link']['yaw']}"
+      fps="30"
+      width="800"
+      height="400"
+      fov="1.3"
+    />
+    <xacro:monocular_camera_macro
+      name="camera9/camera"
+      parent="sensor_kit_base_link"
+      namespace=""
+      x="${calibration['sensor_kit_base_link']['camera9/camera_link']['x']}"
+      y="${calibration['sensor_kit_base_link']['camera9/camera_link']['y']}"
+      z="${calibration['sensor_kit_base_link']['camera9/camera_link']['z']}"
+      roll="${calibration['sensor_kit_base_link']['camera9/camera_link']['roll']}"
+      pitch="${calibration['sensor_kit_base_link']['camera9/camera_link']['pitch']}"
+      yaw="${calibration['sensor_kit_base_link']['camera9/camera_link']['yaw']}"
+      fps="30"
+      width="800"
+      height="400"
+      fov="1.3"
+    />
+    <xacro:monocular_camera_macro
+      name="camera10/camera"
+      parent="sensor_kit_base_link"
+      namespace=""
+      x="${calibration['sensor_kit_base_link']['camera10/camera_link']['x']}"
+      y="${calibration['sensor_kit_base_link']['camera10/camera_link']['y']}"
+      z="${calibration['sensor_kit_base_link']['camera10/camera_link']['z']}"
+      roll="${calibration['sensor_kit_base_link']['camera10/camera_link']['roll']}"
+      pitch="${calibration['sensor_kit_base_link']['camera10/camera_link']['pitch']}"
+      yaw="${calibration['sensor_kit_base_link']['camera10/camera_link']['yaw']}"
       fps="30"
       width="800"

File: aip_xx1_description/urdf/sensors.xacro (robot description, xacro)
@@ -14,5 +14,5 @@
     yaw="${calibration['base_link']['sensor_kit_base_link']['yaw']}"
   />
-  <!-- embedded sensors -->
+  <!-- embedded lidar sensors -->
   <xacro:include filename="$(find velodyne_description)/urdf/VLP-16.urdf.xacro"/>
   <xacro:VLP-16
@@ -33,36 +33,86 @@
     />
   </xacro:VLP-16>
-  <xacro:include filename="$(find livox_description)/urdf/livox_horizon.xacro"/>
-  <xacro:livox_horizon_macro
-    name="livox_front_left"
+  <xacro:include filename="$(find pandar_description)/urdf/pandar_xt32.xacro"/>
+  <xacro:PandarXT-32
+    name="hesai_front_left"
     parent="base_link"
-    x="${calibration['base_link']['livox_front_left_base_link']['x']}"
-    y="${calibration['base_link']['livox_front_left_base_link']['y']}"
-    z="${calibration['base_link']['livox_front_left_base_link']['z']}"
-    roll="${calibration['base_link']['livox_front_left_base_link']['roll']}"
-    pitch="${calibration['base_link']['livox_front_left_base_link']['pitch']}"
-    yaw="${calibration['base_link']['livox_front_left_base_link']['yaw']}"
+    x="${calibration['base_link']['hesai_front_left_base_link']['x']}"
+    y="${calibration['base_link']['hesai_front_left_base_link']['y']}"
+    z="${calibration['base_link']['hesai_front_left_base_link']['z']}"
+    roll="${calibration['base_link']['hesai_front_left_base_link']['roll']}"
+    pitch="${calibration['base_link']['hesai_front_left_base_link']['pitch']}"
+    yaw="${calibration['base_link']['hesai_front_left_base_link']['yaw']}"
   />
-  <xacro:livox_horizon_macro
-    name="livox_front_right"
+  <xacro:PandarXT-32
+    name="hesai_front_right"
     parent="base_link"
-    x="${calibration['base_link']['livox_front_right_base_link']['x']}"
-    y="${calibration['base_link']['livox_front_right_base_link']['y']}"
-    z="${calibration['base_link']['livox_front_right_base_link']['z']}"
-    roll="${calibration['base_link']['livox_front_right_base_link']['roll']}"
-    pitch="${calibration['base_link']['livox_front_right_base_link']['pitch']}"
-    yaw="${calibration['base_link']['livox_front_right_base_link']['yaw']}"
+    x="${calibration['base_link']['hesai_front_right_base_link']['x']}"
+    y="${calibration['base_link']['hesai_front_right_base_link']['y']}"
+    z="${calibration['base_link']['hesai_front_right_base_link']['z']}"
+    roll="${calibration['base_link']['hesai_front_right_base_link']['roll']}"
+    pitch="${calibration['base_link']['hesai_front_right_base_link']['pitch']}"
+    yaw="${calibration['base_link']['hesai_front_right_base_link']['yaw']}"
   />
-  <!-- radar -->
-  <xacro:include filename="$(find aip_xx1_description)/urdf/radar.xacro"/>
+  <!-- embedded radar sensors -->
+  <xacro:include filename="$(find radar_description)/urdf/radar.xacro"/>
   <xacro:radar_macro
-    name="ars408_front_center"
+    name="ars548_front_center"
     parent="base_link"
-    x="${calibration['base_link']['ars408_front_center']['x']}"
-    y="${calibration['base_link']['ars408_front_center']['y']}"
-    z="${calibration['base_link']['ars408_front_center']['z']}"
-    roll="${calibration['base_link']['ars408_front_center']['roll']}"
-    pitch="${calibration['base_link']['ars408_front_center']['pitch']}"
-    yaw="${calibration['base_link']['ars408_front_center']['yaw']}"
+    x="${calibration['base_link']['ars548_front_center_base_link']['x']}"
+    y="${calibration['base_link']['ars548_front_center_base_link']['y']}"
+    z="${calibration['base_link']['ars548_front_center_base_link']['z']}"
+    roll="${calibration['base_link']['ars548_front_center_base_link']['roll']}"
+    pitch="${calibration['base_link']['ars548_front_center_base_link']['pitch']}"
+    yaw="${calibration['base_link']['ars548_front_center_base_link']['yaw']}"
+  />
+  <xacro:radar_macro
+    name="ars548_front_right"
+    parent="base_link"
+    x="${calibration['base_link']['ars548_front_right_base_link']['x']}"
+    y="${calibration['base_link']['ars548_front_right_base_link']['y']}"
+    z="${calibration['base_link']['ars548_front_right_base_link']['z']}"
+    roll="${calibration['base_link']['ars548_front_right_base_link']['roll']}"
+    pitch="${calibration['base_link']['ars548_front_right_base_link']['pitch']}"
+    yaw="${calibration['base_link']['ars548_front_right_base_link']['yaw']}"
+  />
+  <xacro:radar_macro
+    name="ars548_front_left"
+    parent="base_link"
+    x="${calibration['base_link']['ars548_front_left_base_link']['x']}"
+    y="${calibration['base_link']['ars548_front_left_base_link']['y']}"
+    z="${calibration['base_link']['ars548_front_left_base_link']['z']}"
+    roll="${calibration['base_link']['ars548_front_left_base_link']['roll']}"
+    pitch="${calibration['base_link']['ars548_front_left_base_link']['pitch']}"
+    yaw="${calibration['base_link']['ars548_front_left_base_link']['yaw']}"
+  />
+  <xacro:radar_macro
+    name="ars548_back_center"
+    parent="base_link"
+    x="${calibration['base_link']['ars548_back_center_base_link']['x']}"
+    y="${calibration['base_link']['ars548_back_center_base_link']['y']}"
+    z="${calibration['base_link']['ars548_back_center_base_link']['z']}"
+    roll="${calibration['base_link']['ars548_back_center_base_link']['roll']}"
+    pitch="${calibration['base_link']['ars548_back_center_base_link']['pitch']}"
+    yaw="${calibration['base_link']['ars548_back_center_base_link']['yaw']}"
+  />
+  <xacro:radar_macro
+    name="ars548_back_right"
+    parent="base_link"
+    x="${calibration['base_link']['ars548_back_right_base_link']['x']}"
+    y="${calibration['base_link']['ars548_back_right_base_link']['y']}"
+    z="${calibration['base_link']['ars548_back_right_base_link']['z']}"
+    roll="${calibration['base_link']['ars548_back_right_base_link']['roll']}"
+    pitch="${calibration['base_link']['ars548_back_right_base_link']['pitch']}"
+    yaw="${calibration['base_link']['ars548_back_right_base_link']['yaw']}"
+  />
+  <xacro:radar_macro
+    name="ars548_back_left"
+    parent="base_link"
+    x="${calibration['base_link']['ars548_back_left_base_link']['x']}"
+    y="${calibration['base_link']['ars548_back_left_base_link']['y']}"
+    z="${calibration['base_link']['ars548_back_left_base_link']['z']}"
+    roll="${calibration['base_link']['ars548_back_left_base_link']['roll']}"
+    pitch="${calibration['base_link']['ars548_back_left_base_link']['pitch']}"
+    yaw="${calibration['base_link']['ars548_back_left_base_link']['yaw']}"
   />
 </robot>
